Commit message: Initial commit

File: description/ros2_control/diffbot.ros2_control.xacro (robot description, xacro)
@@ -6,6 +6,6 @@
         <plugin>diffdrive_ros2_control/DiffDriveSystemHardware</plugin>
         <param name="loop_rate">30</param>
-        <param name="device_name">zlac8015</param>
-        <param name="port">/dev/zlac8015</param>
+        <param name="device_name">roboteq</param>
+        <param name="port">/dev/ttyACM0</param>
         <param name="baud_rate">115200</param>
         <param name="timeout_ms">25</param>

File: description/urdf/diffbot_description.urdf.xacro (robot description, xacro)
@@ -30,5 +30,5 @@
       <axis xyz="0 1 0" />
       <dynamics damping="0.2" />
-      <limit effort="100" velocity="1.0" />
+      <limit effort="100" velocity="20.0" />
     </joint>
     <joint name="${prefix}right_wheel_joint" type="continuous">
@@ -38,5 +38,5 @@
       <axis xyz="0 1 0" />
       <dynamics damping="0.2" />
-      <limit effort="100" velocity="1.0" />
+      <limit effort="100" velocity="20.0" />
     </joint>
   </xacro:macro>
